File: pcb/right/right.kicad_pcb (KiCad board)
At the start: 2 copper layers, 103 parts, among them SW1 SW_Push, SW10 SW_Push, SW11 SW_Push, SW12 SW_Push, SW13 SW_Push, SW14 SW_Push, SW15 SW_Push, SW16 SW_Push, SW17 SW_Push, SW18 SW_Push, SW19 SW_Push, SW2 SW_Push, SW20 SW_Push, SW21 SW_Push, SW22 SW_Push, SW23 SW_Push, SW24 SW_Push, SW25 SW_Push, SW26 SW_Push, SW27 SW_Push, SW28 SW_Push, SW29 SW_Push, SW3 SW_Push, SW30 SW_Push, SW31 SW_Push, SW32 SW_Push, SW33 SW_Push, SW34 SW_Push, SW35 SW_Push, SW36 SW_Push, SW37 SW_Push, SW38 SW_Push, SW39 SW_Push, SW4 SW_Push, SW40 SW_Push, SW41 SW_Push, SW42 SW_Push, SW43 SW_Push, SW44 SW_Push, SW45 SW_Push, SW46 SW_Push, SW47 SW_Push, SW48 SW_Push, SW49 SW_Push, SW5 SW_Push, SW50 SW_Push, SW51 SW_Push, SW52 SW_Push, SW6 SW_Push, SW7 SW_Push, SW8 SW_Push, SW9 SW_Push

Commit message: pcb: right: Update Design Rules to JLCPCB
Other:
- net class Default: clearance 0.2 -> 0.4
- rule trace_clearance: 0.2 -> 0.4
- rule via_min_size: 0.4 -> 0.45

Commit message: pcb: right: diodes
Parts:
- D1, D10, D11, D12, D13, D14, D15, D16, D17, D18, D19, D2, D20, D21, D22, D23, D24, D25, D26, D27, D28, D29, D3, D30, D31, D32, D33, D34, D35, D36, D37, D38, D39, D4, D40, D41, D42, D43, D44, D45, D46, D47, D48, D49, D5, D50, D51, D6, D7, D8, D9: moved to B.Cu
- moved D5 409.4 mm to (101.1, 107.1), turned to 90 degrees
- moved D2 400.0 mm to (115.4, 49.9), turned to 90 degrees
- moved D3 396.2 mm to (105.8, 69.0), turned to 90 degrees
- moved D16 383.2 mm to (139.2, 107.1), turned to 90 degrees
- moved D8 381.9 mm to (134.4, 49.9), turned to 90 degrees
- moved D14 374.5 mm to (143.9, 69.0), turned to 90 degrees
- moved D17 374.4 mm to (153.5, 126.1), turned to 90 degrees
- moved D7 368.7 mm to (134.4, 30.9), turned to 90 degrees
- moved D9 353.5 mm to (124.9, 69.0), turned to 90 degrees
- moved D27 333.0 mm to (186.8, 88.0), turned to 90 degrees
- moved D12 328.3 mm to (153.5, 30.9), turned to 90 degrees
- moved D25 324.7 mm to (191.6, 49.9), turned to 90 degrees
- moved D24 323.6 mm to (191.6, 30.9), turned to 90 degrees
- moved D4 317.2 mm to (110.6, 88.0), turned to 90 degrees
- moved D11 299.3 mm to (120.1, 107.1), turned to 90 degrees
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