File: pcb/left/left.kicad_pcb (KiCad board)
At the start: 2 copper layers, 101 parts, among them J1 To Right Part, SW1 SW_Push, SW10 L SHIFT, SW11 SW_Push, SW12 SW_Push, SW13 SW_Push, SW14 SW_Push, SW15 SUPER, SW16 SW_Push, SW17 SW_Push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

Commit message: pcb: left: JLCPCB design rules
Other:
- net class Default: clearance 0.2 -> 0.5
- net class Power added: clearance 0.5, trace_width 0.5, via_dia 0.8, via_drill 0.4
- rule trace_clearance: 0.2 -> 0.5
