File: pcb/slash_left/slash_left.kicad_pcb (KiCad board)
At the start: 2 copper layers, 141.8 x 127 mm, 78 parts, among them J1 RJ12, SW1 SW_Push_45deg, SW10 SW_Push_45deg, SW11 SW_Push_45deg, SW12 SW_Push_45deg, SW13 SW_Push_45deg, SW14 SW_Push_45deg, SW15 SW_Push_45deg, SW16 SW_Push_45deg, SW17 SW_Push_45deg, SW18 SW_Push_45deg, SW19 SW_Push_45deg, SW2 SW_Push_45deg, SW20 SW_Push_45deg, SW21 SW_Push_45deg, SW22 SW_Push_45deg, SW23 SW_Push_45deg, SW24 SW_Push_45deg, SW25 SW_Push_45deg, SW26 SW_Push_45deg, SW27 SW_Push_45deg, SW28 SW_Push_45deg, SW29 SW_Push_45deg, SW3 SW_Push_45deg, SW30 SW_Push_45deg, SW31 SW_Push_45deg, SW32 SW_Push_45deg, SW33 SW_Push_45deg, SW34 SW_Push_45deg, SW35 SW_Push_45deg, SW4 SW_Push_45deg, SW5 SW_Push_45deg, SW6 SW_Push_45deg, SW7 SW_Push_45deg, SW8 SW_Push_45deg, SW9 SW_Push_45deg, U1 MCP23018_SO

Commit message: pcb: slash: left: finish
Parts:
- moved D6 21.9 mm to (131.4, 26.5), turned to 0 degrees
- moved C1 1.53 mm to (130.0, 33.2), turned to 180 degrees
Connections:
- U1 pad 10: /COL11 -> Net-(D37-Pad1)
- U1 pad 20: Net-(D37-Pad1) -> /COL5
- U1 pad 21: /ROW0 -> /COL11
- U1 pad 22: /ROW1 -> /COL10
- U1 pad 23: /ROW2 -> /COL9
- U1 pad 24: /COL0 -> /COL8
- U1 pad 25: /COL1 -> /COL7
- U1 pad 26: /COL2 -> /COL6
- U1 pad 27: /COL3 -> /COL4
- U1 pad 3: /COL4 -> /ROW0
- U1 pad 4: /COL5 -> /ROW1
- U1 pad 5: /COL6 -> /ROW2
- U1 pad 6: /COL7 -> /COL0
- U1 pad 7: /COL8 -> /COL1
- U1 pad 8: /COL9 -> /COL2
- U1 pad 9: /COL10 -> /COL3
Routing:
- net /ROW2: track 223.0 -> 367.8 mm, vias 0 -> 2
- net /ROW1: track 285.7 -> 407.2 mm
- net Net-(D37-Pad1): track 0.00 -> 50.6 mm, vias 0 -> 3
- net /COL1: track 96.1 -> 130.8 mm
- net /COL0: track 124.5 -> 152.3 mm
- net /ROW0: track 293.0 -> 317.6 mm
- net /COL5: track 26.2 -> 47.6 mm, vias 3 -> 4
- net +5V: track 59.0 -> 79.1 mm, vias 1 -> 2
- net /COL3: track 78.3 -> 96.2 mm
- net Net-(D6-Pad2): track 0.00 -> 17.4 mm
- net /COL2: track 96.5 -> 113.0 mm
- net Net-(R2-Pad1): track 0.00 -> 12.7 mm, vias 0 -> 1
- net Net-(R3-Pad1): track 0.00 -> 7.86 mm, vias 0 -> 1
- net /COL4: track 58.4 -> 62.1 mm
- net /COL10: track 97.7 -> 100.7 mm, vias 3 -> 4
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
Commit message: pcb: slash: Silkscreen adjustment for production
Other:
- board text added: "19/12/2021"
- board text added: "JLCJLCJLCJLC"
- board text added: "Slash v1 (Left)"
